File: XT-IDE.sch (KiCad schematic (older format))
At the start: 44 parts, among them J1 CONN_3, J2 CONN_3, J3 CONN_2, J4 CONN_2, J5 INTERRUPT, P6 CONN_1, P7 CONN_1, SW1 I/O ADDR, SW2 ROM OPT, U1 74LS573, U10 74LS688, U11 74LS245, U2 74LS573, U3 74LS245, U4 74LS04, U5 74LS32, U6 74LS04, U7 74LS138, U8 74LS688, U9 28C256

Commit message: Silk layer fixes.
Now showing calues of bypass caps and resistors
Parts:
- BUS1: symbol BUSPC -> XT-IDE-rescue:BUSPC
- C1, C10, C11, C2, C3, C4, C5, C6, C7, C8, C9: value C -> 0.1u; symbol C -> XT-IDE-rescue:C
- C12: symbol CP -> XT-IDE-rescue:CP
- D1: symbol LED-RESCUE-XT-IDE -> XT-IDE-rescue:LED-RESCUE-XT-IDE
- IDE1: symbol CONN_20X2 -> XT-IDE-rescue:CONN_20X2
- J1, J2: symbol CONN_3 -> XT-IDE-rescue:CONN_3
- J3, J4: symbol CONN_2 -> XT-IDE-rescue:CONN_2
- J5: symbol CONN_5X2 -> XT-IDE-rescue:CONN_5X2
- P6, P7, TP1, TP2, TP3: symbol CONN_1 -> XT-IDE-rescue:CONN_1
- R1, R2, R3, R4: symbol R -> XT-IDE-rescue:R
- RP1, RP2: symbol RR9 -> XT-IDE-rescue:RR9
- SW1, SW2: symbol DIPS_08 -> XT-IDE-rescue:DIPS_08
- U1, U2: symbol 74LS573 -> XT-IDE-rescue:74LS573
- U10, U8: symbol 74LS688 -> XT-IDE-rescue:74LS688
- U11, U3: symbol 74LS245 -> XT-IDE-rescue:74LS245
- U4, U6: symbol 74LS04 -> XT-IDE-rescue:74LS04
- U5: symbol 74LS32 -> XT-IDE-rescue:74LS32
- U7: symbol 74LS138 -> XT-IDE-rescue:74LS138
- U9: symbol 28C256-RESCUE-XT-IDE -> XT-IDE-rescue:28C256-RESCUE-XT-IDE
Connections:
- wire segments 383 -> 444
